Commit message: working tests

File: src/rrm_simple_robot_model/urdf/arm.urdf (robot description, URDF)
Before this commit: robot arm, 6 links, 5 joints
Links:
- added link link_4; visual cylinder length=0.05 radius=0.01
- added link link_5; visual cylinder length=0.15 radius=0.01
- added link link_6; visual cylinder length=0.1 radius=0.01
Joints:
- removed joint joint_3-tool0
- added joint joint_4: type revolute, parent link_3, child link_4, origin xyz=0 0 0.203 rpy=0 0 0, axis 0 0 1, limit lower=-3.14 upper=3.14 effort=1000.0 velocity=0.5
- added joint joint_5: type revolute, parent link_4, child link_5, origin xyz=0 0 0 rpy=0 0 0, axis 0 1 0, limit lower=-2.2 upper=2.2 effort=1000.0 velocity=0.5
- added joint joint_6: type prismatic, parent link_5, child link_6, origin xyz=0 0 0 rpy=0 0 0, axis 0 0 1, limit lower=0 upper=0.1 effort=1000.0 velocity=0.1
- added joint joint_6-tool0: type fixed, parent link_6, child tool0, origin xyz=0 0 0 rpy=0 0 0

Commit message: working robot mode

File: src/rrm_simple_robot_model/urdf/arm.urdf (robot description, URDF)
Before this commit: robot arm, 9 links, 8 joints
Links:
- removed link link_2_3
- link base_link: geometry visual cylinder length=0.01 radius=0.1
- link tool0: geometry visual box size=0.03 0.03 0.06
Joints:
- removed joint joint_2_3
- removed joint joint_6-tool0
- added joint joint_3-tool0: type fixed, parent link_6, child tool0, origin xyz=0 0 0.1 rpy=0 0 0
- joint joint_3: origin xyz=0 0 0.203 rpy=0 0 0 -> xyz=0 0 0.178 rpy=0 0 0
- joint joint_5: origin xyz=0 0 0 rpy=0 0 0 -> xyz=0 0 0.05 rpy=0 0 0
- joint joint_6: axis 0 0 1 -> 0 1 0; limit lower=0 upper=0.1 effort=1000.0 velocity=0.1 -> lower=0 upper=0.1 effort=1000.0 velocity=0.5; origin xyz=0 0 0 rpy=0 0 0 -> xyz=0 0 0.15 rpy=0 0 0

Commit message: working

File: src/rrm_simple_robot_model/urdf/arm.urdf (robot description, URDF)
Before this commit: robot arm, 8 links, 7 joints
Links:
- link tool0: geometry visual box size=0.02 0.02 0.06
Joints:
- joint joint_6: axis 0 1 0 -> 0 0 1
